File: KiCad/iSpindel-smd/iSpindelPCBv2.kicad_pcb (KiCad board)
At the start: 2 copper layers, 46 x 25 mm, 20 parts, among them J1 PROG, J2 PROG_con, SW1 SW_DPDT_x2, U1 MIC5219-3.3, U2 GY-521, U3 TP4056-shield-6PIN, U4 DS18B20, U5 LoRa_Ra-02, U6 ESP-07S

Commit message: small fix
Parts:
- moved U3 1.00 mm to (158.5, 78.5)
Changed lines of the file:
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@@
-(kicad_pcb (version 4) (host pcbnew 4.0.7)
+(kicad_pcb (version 4) (host pcbnew 4.0.6)
   (general
     (links 51)
     (no_connects 51)
-    (area 125.924999 65.924999 172.075001 91.075001)
+    (area 124.275 60.05 176.025001 92.938095)
     (thickness 1.6)
     (drawings 6)
@@
   )
   (module TP4056-shield-6PIN (layer B.Cu)
-    (at 157.5 78.5 180)
+    (at 158.5 78.5 180)
     (fp_text reference U3 (at 0.5 0 180) (layer B.SilkS)
       (effects (font (size 1 1) (thickness 0.15)) (justify mirror))
@@
       (effects (font (size 1 1) (thickness 0.15)) (justify mirror))
     )
-    (fp_line (start -14 -4) (end -9.5 -4) (layer B.SilkS) (width 0.15))
-    (fp_line (start -9.5 -4) (end -9.5 4) (layer B.SilkS) (width 0.15))
-    (fp_line (start -9.5 4) (end -14.5 4) (layer B.SilkS) (width 0.15))
-    (fp_line (start -14.5 4) (end -14.5 -4) (layer B.SilkS) (width 0.15))
-    (fp_line (start -14.5 -4) (end -14 -4) (layer B.SilkS) (width 0.15))
+    (fp_line (start -14.5 -4) (end -9.5 -4) (layer B.Fab) (width 0.15))
+    (fp_line (start 13 6) (end 13 -6) (layer B.SilkS) (width 0.15))
+    (fp_line (start 13 6) (end 14.5 6) (layer B.SilkS) (width 0.15))
+    (fp_line (start 14.5 6) (end 14.5 8.5) (layer B.SilkS) (width 0.15))
+    (fp_line (start 14.5 8.5) (end 13.5 8.5) (layer B.SilkS) (width 0.15))
+    (fp_line (start 13 -6) (end 14.5 -6) (layer B.SilkS) (width 0.15))
+    (fp_line (start 14.5 -6) (end 14.5 -8.5) (layer B.SilkS) (width 0.15))
+    (fp_line (start 14.5 -8.5) (end 13.5 -8.5) (layer B.SilkS) (width 0.15))
+    (fp_line (start -9.5 -4) (end -9.5 4) (layer B.Fab) (width 0.15))
+    (fp_line (start -9.5 4) (end -14.5 4) (layer B.Fab) (width 0.15))
+    (fp_line (start -14.5 4) (end -14.5 -4) (layer B.Fab) (width 0.15))
     (fp_line (start -13.5 -8.5) (end -13.5 8.5) (layer B.SilkS) (width 0.15))
     (fp_line (start -13.5 8.5) (end 13.5 8.5) (layer B.SilkS) (width 0.15))
-    (fp_line (start 13.5 8.5) (end 13.5 -8.5) (layer B.SilkS) (width 0.15))
     (fp_line (start 13.5 -8.5) (end -13.5 -8.5) (layer B.SilkS) (width 0.15))
-    (pad 3 thru_hole oval (at 10.5 7 180) (size 5 2) (drill 1) (layers *.Cu *.Mask)
+    (pad 3 thru_hole oval (at 11.1 7 180) (size 3 2) (drill 1) (layers *.Cu *.Mask)
       (net 20 "Net-(SW1-Pad2)"))
-    (pad 4 thru_hole oval (at 10.5 -7 180) (size 5 2) (drill 1) (layers *.Cu *.Mask)
+    (pad 4 thru_hole oval (at 11.1 -7 180) (size 3 2) (drill 1) (layers *.Cu *.Mask)
       (net 10 "Net-(U3-Pad4)"))
-    (pad 2 thru_hole oval (at -11.5 -7 180) (size 5 2) (drill 1) (layers *.Cu *.Mask)
+    (pad 2 thru_hole oval (at -11.5 -7 180) (size 3 2) (drill 1) (layers *.Cu *.Mask)
       (net 1 GND))
-    (pad 1 thru_hole oval (at -11.5 7 180) (size 5 2) (drill 1) (layers *.Cu *.Mask)
+    (pad 1 thru_hole oval (at -11.5 7 180) (size 3 2) (drill 1) (layers *.Cu *.Mask)
       (net 11 "Net-(U3-Pad1)"))
   )
