File: KiCad/mergedForOrder/merged2PCBs.kicad_pcb (KiCad board)
At the start: 2 copper layers, 81.5 x 81 mm, 98 parts, among them J1 PROG, J2 PROG_con, SW1 SW_SPDT, SW2 SW_SPDT, U1 GY-521, U1 MIC5219-3.3, U2 GY-521, U2 LoRa_Ra-02, U3 TP4056-shield-6PIN, U3 WeMos_mini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

Commit message: Add led
Parts:
- added C1: 2.2uf, Capacitors_SMD:C_0805, F.Cu at (53.3, 85.3)
- added C2: 470p, Capacitors_SMD:C_0603, F.Cu at (50.1, 85.8)
- added C3: 2.2uf, Capacitors_SMD:C_0805, F.Cu at (53.3, 90.8)
- added C4: 100n, Capacitors_SMD:C_0603, F.Cu at (50.7, 92.9)
- added C5: 10uf, Capacitors_SMD:C_0805, F.Cu at (50.6, 94.6)
- added D1: Schottky, Diodes_SMD:D_SOD-523, F.Cu at (53.4, 113.7)
- added J1: PROG, Pin_Headers:Pin_Header_Straight_1x02_Pitch2.54mm, F.Cu at (42.1, 88.9)
- added J2: PROG_con, Pin_Headers:Pin_Header_Straight_1x04_Pitch2.54mm, F.Cu at (39.6, 85.7)
- added R1: 47K, Resistors_SMD:R_0603, F.Cu at (38.6, 113.7)
- added R2: 4.7k, Resistors_SMD:R_0603, F.Cu at (42.2, 94.6)
- added R3: 10K, Resistors_SMD:R_0603, F.Cu at (44.3, 94.2)
- added R4: 10K, Resistors_SMD:R_0603, F.Cu at (47.0, 93.1)
- added R5: 10K, Resistors_SMD:R_0603, F.Cu at (47.0, 94.7)
- added R6: 10K, Resistors_SMD:R_0603, F.Cu at (38.9, 91.1)
- added R7: 10K, Resistors_SMD:R_0603, F.Cu at (44.9, 89.7)
- added REF**: MountingHole_3.2mm_M3, Mounting_Holes:MountingHole_3.2mm_M3, F.Cu at (56.5, 111.0)
- added REF**: MountingHole_3.2mm_M3, Mounting_Holes:MountingHole_3.2mm_M3, F.Cu at (46.5, 83.5)
- added REF**: MountingHole_3.2mm_M3, Mounting_Holes:MountingHole_3.2mm_M3, F.Cu at (46.5, 81.5)
- added REF**: MountingHole_3.2mm_M3, Mounting_Holes:MountingHole_3.2mm_M3, F.Cu at (45.5, 81.5)
- added REF**: MountingHole_3.2mm_M3, Mounting_Holes:MountingHole_3.2mm_M3, F.Cu at (56.5, 112.0)
- added REF**: MountingHole_3.2mm_M3, Mounting_Holes:MountingHole_3.2mm_M3, F.Cu at (59.5, 112.0)
- added REF**: MountingHole_3.2mm_M3, Mounting_Holes:MountingHole_3.2mm_M3, F.Cu at (59.5, 111.0)
- added REF**: MountingHole_3.2mm_M3, Mounting_Holes:MountingHole_3.2mm_M3, F.Cu at (59.5, 95.5)
- added REF**: MountingHole_3.2mm_M3, Mounting_Holes:MountingHole_3.2mm_M3, F.Cu at (59.5, 96.5)
- added REF**: MountingHole_3.2mm_M3, Mounting_Holes:MountingHole_3.2mm_M3, F.Cu at (56.5, 96.5)
- added REF**: MountingHole_3.2mm_M3, Mounting_Holes:MountingHole_3.2mm_M3, F.Cu at (56.5, 95.5)
- added REF**: MountingHole_3.2mm_M3, Mounting_Holes:MountingHole_3.2mm_M3, F.Cu at (45.5, 83.5)
- added SW1: SW_SPDT, KiCadCustomLibs:SK12D07VG3, F.Cu at (46.5, 115.8)
- added U1: MIC5219-3.3, TO_SOT_Packages_SMD:SOT-23-5, F.Cu at (53.3, 88.1)
- added U3: TP4056-shield-6PIN, KiCadCustomLibs:TP4056-shield-6PIN, B.Cu at (46.5, 104.5)
- added U4: DS18B20, TO_SOT_Packages_THT:TO-92_Inline_Narrow_Oval, F.Cu at (49.8, 89.9)
- added U6: ESP-07S, KiCadCustomLibs:ESP-07S, F.Cu at (46.5, 104.2)
Routing:
- net GND: track 393.8 -> 470.5 mm, vias 122 -> 154
- net VCC: track 81.8 -> 140.8 mm, vias 0 -> 4
- net +3V3: track 223.6 -> 257.8 mm
- net Net-(R1-Pad2): track 23.4 -> 55.7 mm, vias 2 -> 4
- net /VCC_PROG: track 33.1 -> 64.3 mm
- net /Temp: track 205.5 -> 235.2 mm, vias 6 -> 7
- net Net-(J2-Pad2): track 9.74 -> 39.2 mm, vias 0 -> 1
- net Net-(J2-Pad3): track 6.39 -> 34.2 mm, vias 1 -> 2
- net Net-(SW1-Pad3): track 24.8 -> 49.2 mm
- net Net-(D1-Pad2): track 39.0 -> 62.5 mm, vias 3 -> 5
- net /PROG: track 0.00 -> 20.0 mm, vias 0 -> 1
- net /EN: track 14.0 -> 32.2 mm
- net /RES: track 143.3 -> 156.9 mm, vias 4 -> 6
- net Net-(R6-Pad2): track 0.00 -> 13.0 mm, vias 0 -> 2
- net Net-(C2-Pad1): track 1.98 -> 6.00 mm
Other:
- board size 81.5 x 81 mm -> 81.5 x 85 mm
- net class Default: trace_width 0.4 -> 0.3
- net class VCC removed
- rule pad_to_mask_clearance: 0.15 -> 0.1
